File: hardware/electronics/input_protection/input_protection.kicad_sch (KiCad schematic)
At the start: 48 parts, among them J1 PJ-102AH, J2 Header2, J3 Header2, J4 Header3, J5 Header2, J6 Header3, Q1 PSMN012-100YS,115, Q2 BSS138-7-F, Q3 DMN2056U-7, U1 TPS26630RGER, U2 TPS7A1601DGNR, U3 TLV7011DBVR

Commit message: Preserve local hardware work before Git reconciliation
Backup snapshot; hardware development remains in progress.
Parts:
- C5: value 100nF 16V X7R -> 330nF 16V X7R
- J1: footprint Connector_BarrelJack:BarrelJack_CUI_PJ-102AH_Horizontal -> RMX_Input:PJ102AH_RearEdge_E23
- R7: value 6.49k 0.1% 10ppm -> 5.62k 0.1% 10ppm
- S1: footprint Button_Switch_SMD:SW_SPDT_CK_JS102011SAQN -> RMX_Input:JS102011SAQN_RearEdge_E23
Other:
- note added: "Conditional E16/E21 circuit with E23 PCB and A07 housing bounds. No IEC surge or physical startup/fault/assembly validation. Independent final rail disconnects remain separate."
- note removed: "Conditional schematic prototype. No IEC surge claim, PCB/enclosure placement or physical startup/fault validation. Final analog/digital rail OV disconnects remain open."
Changed lines of the file:
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@@
 (kicad_sch (version 20250114) (generator eeschema) (paper "User" 594 470)
-(title_block (title "Standalone RMX - DC input protection / fast OV") (rev "E16") (comment 1 "Schematic prototype; no routed board or bench validation"))
+(title_block (title "Standalone RMX - DC input protection / fast OV") (rev "E16/E21") (comment 1 "Candidate circuit and E23 PCB; no bench validation"))
 (symbol (lib_id "RMX_E15:E15_J1") (at 59.69 139.7 0) (unit 1) (in_bom yes) (on_board yes) (dnp no)
 (property "Reference" "J1" (at 59.69 128.27 0) (effects (font (size 1.27 1.27)) ))
 (property "Value" "PJ-102AH" (at 59.69 151.13 0) (effects (font (size 1.27 1.27)) ))
-(property "Footprint" "Connector_BarrelJack:BarrelJack_CUI_PJ-102AH_Horizontal" (at 59.69 139.7 0) (effects (font (size 1.27 1.27)) (hide yes)))
+(property "Footprint" "RMX_Input:PJ102AH_RearEdge_E23" (at 59.69 139.7 0) (effects (font (size 1.27 1.27)) (hide yes)))
 (property "Datasheet" "https://www.sameskydevices.com/product/resource/pj-102ah.pdf" (at 59.69 139.7 0) (effects (font (size 1.27 1.27)) (hide yes)))
 (pin "1")
@@
 (symbol (lib_id "RMX_E15:E15_R7") (at 123.19 279.4 0) (unit 1) (in_bom yes) (on_board yes) (dnp no)
 (property "Reference" "R7" (at 123.19 270.51 0) (effects (font (size 1.27 1.27)) ))
-(property "Value" "6.49k 0.1% 10ppm" (at 123.19 288.29 0) (effects (font (size 1.27 1.27)) ))
+(property "Value" "5.62k 0.1% 10ppm" (at 123.19 288.29 0) (effects (font (size 1.27 1.27)) ))
 (property "Footprint" "Resistor_SMD:R_0805_2012Metric" (at 123.19 279.4 0) (effects (font (size 1.27 1.27)) (hide yes)))
 (property "Datasheet" "" (at 123.19 279.4 0) (effects (font (size 1.27 1.27)) (hide yes)))
@@
 (symbol (lib_id "RMX_E15:E15_C5") (at 123.19 359.41 0) (unit 1) (in_bom yes) (on_board yes) (dnp no)
 (property "Reference" "C5" (at 123.19 350.52 0) (effects (font (size 1.27 1.27)) ))
-(property "Value" "100nF 16V X7R" (at 123.19 368.3 0) (effects (font (size 1.27 1.27)) ))
+(property "Value" "330nF 16V X7R" (at 123.19 368.3 0) (effects (font (size 1.27 1.27)) ))
 (property "Footprint" "Capacitor_SMD:C_0805_2012Metric" (at 123.19 359.41 0) (effects (font (size 1.27 1.27)) (hide yes)))
 (property "Datasheet" "" (at 123.19 359.41 0) (effects (font (size 1.27 1.27)) (hide yes)))
@@
 (property "Reference" "S1" (at 389.89 146.05 0) (effects (font (size 1.27 1.27)) ))
 (property "Value" "JS102011SAQN" (at 389.89 163.83 0) (effects (font (size 1.27 1.27)) ))
-(property "Footprint" "Button_Switch_SMD:SW_SPDT_CK_JS102011SAQN" (at 389.89 154.94 0) (effects (font (size 1.27 1.27)) (hide yes)))
+(property "Footprint" "RMX_Input:JS102011SAQN_RearEdge_E23" (at 389.89 154.94 0) (effects (font (size 1.27 1.27)) (hide yes)))
 (property "Datasheet" "https://www.ckswitches.com/media/1422/js.pdf" (at 389.89 154.94 0) (effects (font (size 1.27 1.27)) (hide yes)))
 (pin "1")
@@
 (label "VIN_IC" (at 111.76 459.74 0) (effects (font (size 1 1)) (justify left bottom)))
 (text "E16: E15 DC inlet/eFuse + independent TLV7011 fast OV shutdown. Auxiliary supply powers comparison and PGOOD guard; no MCU or main-rail dependency." (at 20.32 20.32 0) (effects (font (size 1.27 1.27)) (justify left)))
-(text "Conditional schematic prototype. No IEC surge claim, PCB/enclosure placement or physical startup/fault validation. Final analog/digital rail OV disconnects remain open." (at 20.32 30.48 0) (effects (font (size 1.27 1.27)) (justify left)))
+(text "Conditional E16/E21 circuit with E23 PCB and A07 housing bounds. No IEC surge or physical startup/fault/assembly validation. Independent final rail disconnects remain separate." (at 20.32 30.48 0) (effects (font (size 1.27 1.27)) (justify left)))
 (text "FAST_OV_OUT high -> Q3 grounds POWER_RUN/SHDN. R17 provides hysteresis. Local wiring, comparator delay/drive and transferred fault charge require qualification." (at 20.32 425.45 0) (effects (font (size 1.27 1.27)) (justify left)))
 (text "Auxiliary PG/C10 holds SHDN low during startup. S1 missing -> OFF via47k. AUX starts through external FET body diode before the internal pass FET." (at 20.32 434.34 0) (effects (font (size 1.27 1.27)) (justify left)))
