File: hardware/electronics/power_supply/power_supply.kicad_sch (KiCad schematic)
At the start: 157 parts, among them J1 Header2, J2 Header6, J3 Header2, J4 Header6, J5 Header2, U1 LT3471EDD#PBF, U10 LT3090IDD#PBF, U11 LT3090IDD#PBF, U12 LT1634AIS8-2.5#PBF, U13 LT3471EDD#PBF, U2 TPS62933FDRLR, U3 TPS62933FDRLR, U4 REF5025EIDR, U5 OPA4192ID, U6 OPA2192ID, U7 LT3080IMS8E#PBF, U8 LT3080IQ#PBF, U9 LT3080IMS8E#PBF

Commit message: Preserve local hardware work before Git reconciliation
Backup snapshot; hardware development remains in progress.
Parts:
- C17: value 33nF 16V X7R -> 1uF 16V X7R
- C32, C33: value 1uF film 63V 10% -> 1uF film 63V 10% MKS2C041001F00KSSD
- J4: footprint Connector_PinHeader_2.54mm:PinHeader_1x06_P2.54mm_Vertical -> Connector_PinHeader_2.54mm:PinHeader_2x03_P2.54mm_Vertical
- L1, L6: value 33uH 20% Isat>=3A Irms>=1.5A DCR<=0.2ohm -> 33uH 20% SRP7050WA-330M; footprint Inductor_SMD:L_Bourns_SRP6060FA -> RMX_Power:SRP7050WA
- L2, L3, L7, L8: value 68uH 20% Isat>=3A Irms>=1.5A DCR<=0.2ohm -> 68uH 20% SRP1050WA-680M; footprint Inductor_SMD:L_Bourns_SRP1050WA -> RMX_Power:SRP1050WA
- L4, L5: value 10uH 20% Isat>=6A Irms>=3A DCR<=0.1ohm -> 10uH 20% SRP1050WA-100M; footprint Inductor_SMD:L_Bourns_SRP1050WA -> RMX_Power:SRP1050WA
