File: hardware/electronics/processor_carrier/processor_carrier.kicad_pcb (KiCad board)
At the start: 4 copper layers, 150 x 65 mm, 84 parts, among them J1 Header2, J10 Header4, J11 Header8, J12 Header8, J2 Header5, J20 Header3, J21 Header3, J22 Header3, J23 Header3, J24 Header3, J25 Header3, J26 Header3, J27 Header3, J28 Header3, J29 Header3, J3 Header6, J4 Header5, J5 Header5, J6 Header6, J7 Header2, J8 Header2, J9 Header4, U1 DaisySeed3

Commit message: Preserve local hardware work before Git reconciliation
Backup snapshot; hardware development remains in progress.
Parts:
- moved C6 16.2 mm to (170.0, 148.0)
- moved R3 8.54 mm to (171.0, 131.0)
- moved J12 5.83 mm to (153.0, 123.0), turned to 90 degrees
- moved J11 1.41 mm to (145.0, 119.0)
- moved R4 0.85 mm to (129.2, 141.5)
- moved R11 0.81 mm to (139.3, 141.5)
- moved J20 0.60 mm to (169.0, 157.8)
- moved J21 0.60 mm to (176.5, 157.8)
- moved J22 0.60 mm to (184.0, 157.8)
- moved J23 0.60 mm to (191.5, 157.8)
- moved J24 0.60 mm to (199.0, 157.8)
- moved J25 0.60 mm to (206.5, 157.8)
- moved J26 0.60 mm to (214.0, 157.8)
- moved J27 0.60 mm to (221.5, 157.8)
- moved J28 0.60 mm to (229.0, 157.8)
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Routing:
- net /V3V3_IO: track 0.00 -> 251.5 mm, vias 0 -> 2
- net /ARMED: track 0.00 -> 248.6 mm, vias 0 -> 6
- net /SDA: track 0.00 -> 230.4 mm, vias 0 -> 3
- net /MCU_PERMIT: track 0.00 -> 168.9 mm, vias 0 -> 4
- net /V3V3_ANALOG: track 0.00 -> 159.0 mm, vias 0 -> 2
- net /POT_RAW_09: track 0.00 -> 148.6 mm, vias 0 -> 2
- net /POT_RAW_08: track 0.00 -> 143.6 mm, vias 0 -> 2
- net /POT_RAW_07: track 0.00 -> 138.6 mm, vias 0 -> 2
- net /POT_RAW_06: track 0.00 -> 133.6 mm, vias 0 -> 2
- net /SCL: track 0.00 -> 132.9 mm
- net /POT_RAW_05: track 0.00 -> 128.7 mm, vias 0 -> 2
- net /CODEC_RUN: track 0.00 -> 124.5 mm, vias 0 -> 2
- net /POT_RAW_04: track 0.00 -> 123.9 mm, vias 0 -> 2
- net /POT_RAW_03: track 0.00 -> 118.9 mm, vias 0 -> 2
- net /DAC_DATA: track 0.00 -> 116.6 mm, vias 0 -> 3
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- added copper zone on In1.Cu, net /AGND
