File: hardware/electronics/processor_carrier/processor_carrier.kicad_sch (KiCad schematic)
At the start: 76 parts, among them J1 Header2, J10 Header4, J11 Header8, J12 Header8, J2 Header5, J20 Header3, J21 Header3, J22 Header3, J23 Header3, J24 Header3, J25 Header3, J26 Header3, J27 Header3, J28 Header3, J29 Header3, J3 Header6, J4 Header5, J5 Header5, J6 Header6, J7 Header2, J8 Header2, J9 Header4, U1 DaisySeed3

Commit message: Preserve local hardware work before Git reconciliation
Backup snapshot; hardware development remains in progress.
Other:
- note added: "Routed150x65mm carrier: front-slot Seed and2mm E18 daughterboard shift implemented in PCB/A05 CAD; physical assembly unverified."
- note removed: "Proposed150x65mm carrier: front-slot Seed placement and2mm E18 daughterboard shift still require PCB/CAD implementation."
Changed lines of the file:
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@@
 (text "E19 - external-profile Seed3 processor carrier.40 module pins,10 analog pots,control-hub/codec/relay/LED/sensor/SD interfaces." (at 20 18 0) (effects (font (size 1.27 1.27)) (justify left)))
 (text "3.3V outputs are separate: analog pin21 excites pots; digital pin38 powers shared logic. AGND and DGND join on carrier." (at 20 28 0) (effects (font (size 1.27 1.27)) (justify left)))
-(text "Proposed150x65mm carrier: front-slot Seed placement and2mm E18 daughterboard shift still require PCB/CAD implementation." (at 20 638 0) (effects (font (size 1.27 1.27)) (justify left)))
+(text "Routed150x65mm carrier: front-slot Seed and2mm E18 daughterboard shift implemented in PCB/A05 CAD; physical assembly unverified." (at 20 638 0) (effects (font (size 1.27 1.27)) (justify left)))
 (text "No whole-bus/3.3V load, USB partial-power/backfeed, ADC acquisition/accuracy, SDMMC SI or physical fit approval. No fabrication release." (at 20 648 0) (effects (font (size 1.27 1.27)) (justify left)))
 (embedded_fonts no))
