File: hardware/electronics/rail_disconnect/rail_disconnect.kicad_sch (KiCad schematic)
At the start: 162 parts, among them J1 Header6, J2 Header2, J3 Header6, J4 Header2, J5 Header3, J6 Header3, Q1 CSD18540Q5B, Q10 CSD18510Q5B, Q11 CSD18510Q5B, Q12 CSD18510Q5B, Q2 CSD18540Q5B, Q3 CSD18540Q5B, Q4 CSD18540Q5B, Q5 CSD18540Q5B, Q6 CSD18540Q5B, Q7 CSD18540Q5B, Q8 CSD18540Q5B, Q9 CSD18510Q5B, U1 SI8751AB-ISR, U10 TLV1824IDR, U11 SN74LVC08APWR, U12 SN74LVC08APWR, U2 SI8751AB-ISR, U3 SI8751AB-ISR, U4 SI8751AB-ISR, U5 SI8751AB-ISR, U6 SI8751AB-ISR, U7 REF35125QDBVR, U8 OPA2333AID, U9 TLV1824IDR

Commit message: Preserve local hardware work before Git reconciliation
Backup snapshot; hardware development remains in progress.
Parts:
- added Q13: CSD18510Q5B, Package_SON:VSONP-8-1EP_5x6_P1.27mm, symbol RMX_E17:E17_Q13
- added Q14: CSD18510Q5B, Package_SON:VSONP-8-1EP_5x6_P1.27mm, symbol RMX_E17:E17_Q14
Connections:
- net 5V_DIG: now also Q14.3 (DRAIN_GROUP)
- net 5V_DIG_COMMON: now also Q13.1 (SOURCE_GROUP), Q14.1 (SOURCE_GROUP)
- net 5V_DIG_GATE: now also Q13.2 (GATE_GROUP), Q14.2 (GATE_GROUP)
- net 5V_DIG_SRC: now also Q13.3 (DRAIN_GROUP)
Changed lines of the file:
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@@
 (kicad_sch (version 20250114) (generator eeschema) (paper "User" 1250 1230)
-(title_block (title "Standalone RMX - Rail disconnects / independent OV") (rev "E17") (comment 1 "Schematic prototype; no routed board or bench validation"))
+(title_block (title "Standalone RMX - Rail disconnects / independent OV") (rev "E17/E21") (comment 1 "Schematic prototype; no routed board or bench validation"))
 (symbol (lib_id "RMX_E17:E17_Q1") (at 69.85 69.85 0) (unit 1) (in_bom yes) (on_board yes) (dnp no)
 (property "Reference" "Q1" (at 69.85 60.96 0) (effects (font (size 1.27 1.27)) ))
@@
 (wire (pts (xy 1150.62 849.63) (xy 1155.7 849.63)) (stroke (width 0) (type default)))
 (label "AGND" (at 1155.7 849.63 0) (effects (font (size 1 1)) (justify left bottom)))
+(symbol (lib_id "RMX_E17:E17_Q13") (at 69.85 229.87 0) (unit 1) (in_bom yes) (on_board yes) (dnp no)
+(property "Reference" "Q13" (at 69.85 220.98 0) (effects (font (size 1.27 1.27)) ))
+(property "Value" "CSD18510Q5B" (at 69.85 238.76 0) (effects (font (size 1.27 1.27)) ))
+(property "Footprint" "Package_SON:VSONP-8-1EP_5x6_P1.27mm" (at 69.85 229.87 0) (effects (font (size 1.27 1.27)) (hide yes)))
+(property "Datasheet" "https://www.ti.com/lit/ds/symlink/csd18510q5b.pdf" (at 69.85 229.87 0) (effects (font (size 1.27 1.27)) (hide yes)))
+(pin "1")
+(pin "2")
+(pin "3")
+(instances (project "rail_disconnect" (path "/9e0b98e0-a19b-56f7-a6d3-ac7e00e7a359" (reference "Q13") (unit 1)))))
+(wire (pts (xy 54.61 227.33) (xy 49.53 227.33)) (stroke (width 0) (type default)))
+(label "5V_DIG_COMMON" (at 49.53 227.33 0) (effects (font (size 1 1)) (justify right bottom)))
+(wire (pts (xy 54.61 232.41) (xy 49.53 232.41)) (stroke (width 0) (type default)))
+(label "5V_DIG_GATE" (at 49.53 232.41 0) (effects (font (size 1 1)) (justify right bottom)))
+(wire (pts (xy 85.09 229.87) (xy 90.17 229.87)) (stroke (width 0) (type default)))
+(label "5V_DIG_SRC" (at 90.17 229.87 0) (effects (font (size 1 1)) (justify left bottom)))
+(symbol (lib_id "RMX_E17:E17_Q14") (at 245.11 229.87 0) (unit 1) (in_bom yes) (on_board yes) (dnp no)
+(property "Reference" "Q14" (at 245.11 220.98 0) (effects (font (size 1.27 1.27)) ))
+(property "Value" "CSD18510Q5B" (at 245.11 238.76 0) (effects (font (size 1.27 1.27)) ))
+(property "Footprint" "Package_SON:VSONP-8-1EP_5x6_P1.27mm" (at 245.11 229.87 0) (effects (font (size 1.27 1.27)) (hide yes)))
+(property "Datasheet" "https://www.ti.com/lit/ds/symlink/csd18510q5b.pdf" (at 245.11 229.87 0) (effects (font (size 1.27 1.27)) (hide yes)))
+(pin "1")
+(pin "2")
+(pin "3")
+(instances (project "rail_disconnect" (path "/9e0b98e0-a19b-56f7-a6d3-ac7e00e7a359" (reference "Q14") (unit 1)))))
+(wire (pts (xy 229.87 227.33) (xy 224.79 227.33)) (stroke (width 0) (type default)))
+(label "5V_DIG_COMMON" (at 224.79 227.33 0) (effects (font (size 1 1)) (justify right bottom)))
+(wire (pts (xy 229.87 232.41) (xy 224.79 232.41)) (stroke (width 0) (type default)))
+(label "5V_DIG_GATE" (at 224.79 232.41 0) (effects (font (size 1 1)) (justify right bottom)))
+(wire (pts (xy 260.35 229.87) (xy 265.43 229.87)) (stroke (width 0) (type default)))
+(label "5V_DIG" (at 265.43 229.87 0) (effects (font (size 1 1)) (justify left bottom)))
 (symbol (lib_id "RMX_E17:E17_U7") (at 100.33 449.58 0) (unit 1) (in_bom yes) (on_board yes) (dnp no)
 (property "Reference" "U7" (at 100.33 435.61 0) (effects (font (size 1.27 1.27)) ))
